File: resin-rover.sch (KiCad schematic (older format))
At the start: 42 parts

Commit message: Add 5V and 6V voltage regulators
Parts:
- removed C?: C, symbol C
- added C? (x4): 22u, symbol C
- added C? (x2): 100n, symbol C
- added C? (x2): 8.2n, symbol C
- added C?: 1n, symbol C
- added C?: 27p, symbol C
- added C?: 1.2n, symbol C
- added C?: 30p, symbol C
- added C?: C, symbol C
- added D? (x2): D_Schottky, symbol D_Schottky
- added D? (x2): LED, symbol LED
- added L? (x2): 3.3u, symbol L
- added R? (x2): 10.2K, symbol R
- added R?: 1.56K, symbol R
- added R?: 30.1K, symbol R
- added R?: 1.93K, symbol R
- added R?: 26.7K, symbol R
- added R? (x4): 4.7K, symbol R
- added R? (x2): 1K, symbol R
- added U? (x2): TPS54332DDA, SOIC127P600X170-9N, symbol TPS54332DDA
- C? (x4): value C -> 10u
- C? (x2): value C -> 1u
- C?: value C -> 0.1u
- L?: value L -> 6.8u
- R? (x2): value R -> 0.2
- R?: value R -> 1K
- R? (x2): value R -> 10K
- R?: value R -> 0.1
Connections:
- net labels added: 3.3V, 5V, VSENSE
- wire segments 176 -> 213
- no-connect marks 7 -> 9
Other:
- note added: "5V regulator"
- note added: "6V regulator"
- note added: "RPi header"
- moved on the sheet: C?, D?, J?, L?, Q?, R?, U?

Commit message: Add line following circuit
Parts:
- added C?: 0.1u, symbol C
- added J? (x2): CONN_01X04, symbol CONN_01X04
- added R? (x6): 4.7K, symbol R
- added U? (x3): QRE1113GR, 4LEADSMD, symbol QRE1113GR
- added U?: ADS1015, SOP50P490X110-10N, symbol ADS1015QDGSRQ1
- U? (x2): value DRV8830DGQ -> DRV8830
- U? (x2): value TPS54332DDA -> TPS54332
Connections:
- net 3.3V: now also J?.1 (P1), J?.17 (P17), C?.2, J?.3 (P3), J?.3 (P3), R?.2, R?.2, R?.2, R?.2, R?.2, R?.2, U?.8 (VDD)
- net 5V: now also J?.2 (P2), J?.4 (P4)
- net GND: now also J?.14 (P14), J?.20 (P20), J?.25 (P25), J?.30 (P30), J?.34 (P34), J?.39 (P39), J?.6 (P6), J?.9 (P9), C?.1, J?.4 (P4), J?.4 (P4), U?.1 (ADDR), U?.3 (GND), U?.7 (AIN3), U?.E, U?.E, U?.E, U?.K, U?.K, U?.K
- net RX: now also J?.2 (P2)
- net SCL: now also J?.1 (P1), U?.10 (SCL)
- net SDA: now also J?.2 (P2), U?.9 (SDA)
- net TX: now also J?.1 (P1)
- net VCC: now also C?.2, C?.2, D?.2 (A), U?.2 (VIN)
- new net: R?.1, U?.A (x3)
- new net ADC0: R?.1, U?.4 (AIN0), U?.C
- new net ADC1: R?.1, U?.5 (AIN1), U?.C
- new net ADC2: R?.1, U?.6 (AIN2), U?.C
Other:
- note added: "ADC\n"
- note added: "Center sensor\n"
- note added: "I²C pins"
- note added: "Left sensor\n"
- note added: "Line following circuit"
- note added: "Right sensor\n"
- note added: "UART pins"
- moved on the sheet: C?, D?, J?, R?, U?

Commit message: Add BOM and change battery charger to MP2610
Parts:
- removed C? (x4): 10u, symbol C
- removed C? (x2): 1u, symbol C
- removed C?: 0.1u, symbol C
- removed D?: LED, symbol LED
- removed L?: 6.8u, symbol L
- removed R?: 1K, symbol R
- removed R? (x2): 10K, symbol R
- removed R?: 0.1, symbol R
- removed U?: MP2615, symbol MP2615
- added C10: 0.1u, Capacitors_SMD:C_0805, symbol C
- added C12: 0.1u, Capacitors_SMD:C_0201, symbol C
- added C13, C14: 2.2n, Capacitors_SMD:C_0201, symbol C
- added C15: 22u, Capacitors_SMD:C_0603, symbol C
- added C7: 1u, Capacitors_SMD:C_0805, symbol C
- added C9: 4.7u, Capacitors_SMD:C_0805, symbol C
- added D2, D7: LED, LEDs:LED_0603, symbol LED
- added D6, D8: Schottky, Diodes_SMD:D_SMA_Standard, symbol D_Schottky
- added L1: 6.8u, footprints:SRN6045, symbol L
- added R20: 10K, Resistors_SMD:R_0805, symbol R
- added R21, R22: 1K, Resistors_SMD:R_0402, symbol R
- added R25: 2.49K, Resistors_SMD:R_0603, symbol R
- added R32, R33, R34, R35: 4.7K, Resistors_SMD:R_0402, symbol R
- added R36: 750, Resistors_SMD:R_0603, symbol R
- added R37: 0.1, Resistors_SMD:R_0805, symbol R
- added TH1: NTC 10K, Resistors_SMD:R_0603, symbol Thermistor_NTC
- added U8: MP2610, Housings_DFN_QFN:QFN-16-1EP_4x4mm_Pitch0.65mm, symbol MP2610
- C1, C6: renamed from C?; value C -> 10u; footprint (none) -> Capacitors_SMD:C_0805
- C11, C19, C2, C3, C4, C5, C8: renamed from C?; footprint (none) -> Capacitors_SMD:C_0805
- C16, C17: renamed from C?; footprint (none) -> Capacitors_SMD:C_1210
- C18, C20, C21, C22, C23: renamed from C?; footprint (none) -> Capacitors_SMD:C_0201
- C24, C25: renamed from C?; footprint (none) -> Capacitors_SMD:C_0402
- C26, C27: renamed from C?; footprint (none) -> Capacitors_SMD:C_0603
- D1, D3: renamed from D?; footprint (none) -> LEDs:LED_0603
- D4: renamed from D?; footprint (none) -> Diodes_SMD:D_SOD-123F
- D5: renamed from D?; footprint (none) -> Diodes_SMD:D_SMA_Standard
- J1: renamed from J?; footprint (none) -> Connectors:BARREL_JACK
- J2: renamed from J?; footprint (none) -> Connectors_JST:JST_XH_B03B-XH-A_03x2.50mm_Straight
- J3, J4, J5, J6: renamed from J?; footprint (none) -> Connectors_Phoenix:PhoenixContact_MCV-G_02x3.81mm_Vertical
- J7: renamed from J?; footprint (none) -> Pin_Headers:Pin_Header_Straight_2x20_Pitch2.54mm_SMD
- J8, J9: renamed from J?; footprint (none) -> Pin_Headers:Pin_Header_Angled_1x04_Pitch2.54mm
- L2, L3: renamed from L?; footprint (none) -> footprints:SRN6045
- R1, R10, R13: renamed from R?; value 4.7K -> 100; footprint (none) -> Resistors_SMD:R_0805
- R11, R14, R17, R18, R2, R23, R26, R27, R3: renamed from R?; footprint (none) -> Resistors_SMD:R_0402
- R12, R16, R5: renamed from R?; value 4.7K -> 10K; footprint (none) -> Resistors_SMD:R_0805
- R15, R19, R24, R4: renamed from R?; footprint (none) -> Resistors_SMD:R_0805
- R28: renamed from R?; value 10.2K -> 10K; footprint (none) -> Resistors_SMD:R_0805
- R29: renamed from R?; value 1.56K -> 1.54K; footprint (none) -> Resistors_SMD:R_0805
- R30: renamed from R?; value 10.2K -> 10.5K; footprint (none) -> Resistors_SMD:R_0805
- R31: renamed from R?; value 1.93K -> 2K; footprint (none) -> Resistors_SMD:R_0805
- R6, R7, R8, R9: renamed from R?; footprint (none) -> Resistors_SMD:R_1206
- U7: renamed from U?; footprint (none) -> TO_SOT_Packages_SMD:SOT-23-6
- gave numbers to parts that had none: 10
Connections:
- net 3.3V: now also R32.1, R33.2, R34.2, R35.2
- net 6V: now also C1.1, C6.1, U2.4 (VCC), U6.4 (VCC); no longer C1.2, C6.2
- net CHG_EN: now also U8.6 (EN)
- net GND: now also C1.2, C6.2, R15.2, U9.2 (ALERT/RDY), C12.1, C13.1, C14.1, C15.1, C7.1, C9.2, D8.2 (A), TH1.2, U8.12 (GND), U8.17 (PAD)
- net SCL: now also R32.2, R34.1
- net SDA: now also R33.1, R35.1
- net VCC: now also D6.2 (A)
- net V_BATT: now also C15.2, R37.1, U8.10 (BATT)
- new net: R20.1, TH1.1, U8.1 (NTC)
- new net: L1.1, R37.2, U8.11 (CSP)
- new net: C12.2, U8.13 (TMR)
- new net: C10.2, U8.14 (BST)
- new net: C10.1, D8.1 (K), L1.2, U8.15 (SW)
- new net: C9.1, D6.1 (K), U8.16 (VIN)
- new net: R22.1, U8.2 (ACOK)
- new net: D7.1 (K), U8.3 (CHGOK)
- new net: C7.2, D2.2 (A), R20.2, R21.1, U8.4 (VREF33), U8.7 (CELLS)
- new net: R25.2, U8.8 (COMPV)
- new net: R36.2, U8.9 (COMPI)
- new net: C13.2, R25.1
- new net: C14.2, R36.1
- new net: D7.2 (A), R21.2
- new net: D2.1 (K), R22.2
- no-connect marks 9 -> 30
Other:
- note added: "Headers"
- moved on the sheet: C1, C11, C2, C3, C4, C5, C6, C8, D1, D3, J3, J4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

Commit message: Add layout and fabrication files
Parts:
- removed J8, J9: CONN_01X04, Pin_Headers:Pin_Header_Angled_1x04_Pitch2.54mm, symbol CONN_01X04
- added J10, J11, J12, J13, J14, J15, J8, J9: TEST_1P, Measurement_Points:Measurement_Point_Round-SMD-Pad_Big, symbol TEST_1P
- J2: footprint Connectors_JST:JST_XH_B03B-XH-A_03x2.50mm_Straight -> Connectors_JST:JST_XH_S03B-XH-A_03x2.50mm_Angled
Connections:
- net 3.3V: now also J7.18 (P18), J7.2 (P2); no longer J7.1 (P1), J7.17 (P17)
- net 5V: now also J7.1 (P1), J7.3 (P3), J10.1, J14.1; no longer J7.2 (P2), J7.4 (P4)
- net GND: now also J7.10 (P10), J7.13 (P13), J7.19 (P19), J7.26 (P26), J7.29 (P29), J7.33 (P33), J7.40 (P40), J7.5 (P5), J11.1, J15.1; no longer J7.14 (P14), J7.20 (P20), J7.25 (P25), J7.30 (P30), J7.34 (P34), J7.39 (P39), J7.6 (P6), J7.9 (P9)
- net RX: now also J7.9 (P9), J9.1; no longer J7.10 (P10)
- net SCL: now also J7.6 (P6), J12.1; no longer J7.5 (P5)
- net SDA: now also J7.4 (P4), J13.1; no longer J7.3 (P3)
- net TX: now also J7.7 (P7), J8.1; no longer J7.8 (P8)
- net VSENSE renamed VSENSE_5V
- net VSENSE_5V: no longer R28.1, R29.2, U10.5 (VSENSE)
- new net VSENSE_6V: R28.1, R29.2, U10.5 (VSENSE)
Changed lines of the file:
@@
 F 3 "" H -2050 -600 50  0001 C CNN
 	1    2400 2750
-	1    0    0    -1
+	-1   0    0    -1
 $EndComp
 $Comp
@@
 F 0 "J2" H 3750 14000 50  0000 R CNN
 F 1 "2S LIPO" H 3850 13500 50  0000 R CNN
-F 2 "Connectors_JST:JST_XH_B03B-XH-A_03x2.50mm_Straight" H 500 12000 50  0001 C CNN
-F 3 "B3B-XH-A" H 500 12000 50  0001 C CNN
+F 2 "Connectors_JST:JST_XH_S03B-XH-A_03x2.50mm_Angled" H 500 12000 50  0001 C CNN
+F 3 "S3B-XH-A" H 500 12000 50  0001 C CNN
 	1    3700 13750
 	-1   0    0    -1
@@
 $EndComp
 Text Label 12650 10950 0    60   ~ 0
-VSENSE
+VSENSE_6V
 $Comp
 L GND #PWR09
@@
 6V
 Text Label 15350 11500 0    60   ~ 0
-VSENSE
+VSENSE_6V
 Text Notes 13550 10200 0    60   ~ 12
 6V regulator
@@
 $EndComp
 Text Label 12650 13450 0    60   ~ 0
-VSENSE
+VSENSE_5V
 $Comp
 L GND #PWR010
@@
 5V
 Text Label 15350 14000 0    60   ~ 0
-VSENSE
+VSENSE_5V
 NoConn ~ 13200 13850
 Text Label 16550 7350 0    60   ~ 0
@@
 3.3V
 $Comp
-L CONN_01X04 J8
-U 1 1 58EDAEC2
-P 4450 2650
-F 0 "J8" H 4528 2691 50  0000 L CNN
-F 1 "CONN_01X04" H 4528 2600 50  0000 L CNN
-F 2 "Pin_Headers:Pin_Header_Angled_1x04_Pitch2.54mm" H 700 350 50  0001 C CNN
-F 3 "" H 700 350 50  0001 C CNN
-	1    4450 2650
-	1    0    0    -1
-$EndComp
-$Comp
-L CONN_01X04 J9
-U 1 1 58EDAFF8
-P 6200 2850
-F 0 "J9" H 6278 2891 50  0000 L CNN
-F 1 "CONN_01X04" H 6278 2800 50  0000 L CNN
-F 2 "Pin_Headers:Pin_Header_Angled_1x04_Pitch2.54mm" H 2450 550 50  0001 C CNN
-F 3 "" H 2450 550 50  0001 C CNN
-	1    6200 2850
-	1    0    0    -1
-$EndComp
-$Comp
 L GND #PWR018
 U 1 1 58EDB40A
@@
 $EndComp
 Text Label 4000 2700 0    60   ~ 0
-3.3V
+5V
 Text Label 5750 2900 0    60   ~ 0
-3.3V
+5V
 Text GLabel 5650 2700 0    60   Input ~ 0
 SCL
@@
 Wire Wire Line
 	5350 12050 5350 12200
+$Comp
+L TEST_1P J8
+U 1 1 58F9284E
+P 4250 2500
+F 0 "J8" V 4204 2688 50  0000 L CNN
+F 1 "TEST_1P" V 4200 2850 50  0000 L CNN
+F 2 "Measurement_Points:Measurement_Point_Round-SMD-Pad_Big" H -400 0   50  0001 C CNN
+F 3 "" H -400 0   50  0001 C CNN
+	1    4250 2500
+	0    1    1    0
+$EndComp
+$Comp
+L TEST_1P J9
+U 1 1 58F95589
+P 4250 2600
+F 0 "J9" V 4204 2788 50  0000 L CNN
+F 1 "TEST_1P" V 4200 2950 50  0000 L CNN
+F 2 "Measurement_Points:Measurement_Point_Round-SMD-Pad_Big" H -400 100 50  0001 C CNN
+F 3 "" H -400 100 50  0001 C CNN
+	1    4250 2600
+	0    1    1    0
+$EndComp
+$Comp
+L TEST_1P J10
+U 1 1 58F956BC
+P 4250 2700
+F 0 "J10" V 4204 2888 50  0000 L CNN
+F 1 "TEST_1P" V 4200 3050 50  0000 L CNN
+F 2 "Measurement_Points:Measurement_Point_Round-SMD-Pad_Big" H -400 200 50  0001 C CNN
+F 3 "" H -400 200 50  0001 C CNN
+	1    4250 2700
+	0    1    1    0
+$EndComp
+$Comp
+L TEST_1P J11
+U 1 1 58F957F2
+P 4250 2800
+F 0 "J11" V 4204 2988 50  0000 L CNN
+F 1 "TEST_1P" V 4200 3150 50  0000 L CNN
+F 2 "Measurement_Points:Measurement_Point_Round-SMD-Pad_Big" H -400 300 50  0001 C CNN
+F 3 "" H -400 300 50  0001 C CNN
+	1    4250 2800
+	0    1    1    0
+$EndComp
+$Comp
+L TEST_1P J12
+U 1 1 58F9592F
+P 6000 2700
+F 0 "J12" V 5954 2888 50  0000 L CNN
+F 1 "TEST_1P" V 5950 3050 50  0000 L CNN
+F 2 "Measurement_Points:Measurement_Point_Round-SMD-Pad_Big" H 1350 200 50  0001 C CNN
+F 3 "" H 1350 200 50  0001 C CNN
+	1    6000 2700
+	0    1    1    0
+$EndComp
+$Comp
+L TEST_1P J13
+U 1 1 58F95AC3
+P 6000 2800
+F 0 "J13" V 5954 2988 50  0000 L CNN
+F 1 "TEST_1P" V 5950 3150 50  0000 L CNN
+F 2 "Measurement_Points:Measurement_Point_Round-SMD-Pad_Big" H 1350 300 50  0001 C CNN
+F 3 "" H 1350 300 50  0001 C CNN
+	1    6000 2800
+	0    1    1    0
+$EndComp
+$Comp
+L TEST_1P J14
+U 1 1 58F95C02
+P 6000 2900
+F 0 "J14" V 5954 3088 50  0000 L CNN
+F 1 "TEST_1P" V 5950 3250 50  0000 L CNN
+F 2 "Measurement_Points:Measurement_Point_Round-SMD-Pad_Big" H 1350 400 50  0001 C CNN
+F 3 "" H 1350 400 50  0001 C CNN
+	1    6000 2900
+	0    1    1    0
+$EndComp
+$Comp
+L TEST_1P J15
+U 1 1 58F95D44
+P 6000 3000
+F 0 "J15" V 5954 3188 50  0000 L CNN
+F 1 "TEST_1P" V 5950 3350 50  0000 L CNN
+F 2 "Measurement_Points:Measurement_Point_Round-SMD-Pad_Big" H 1350 500 50  0001 C CNN
+F 3 "" H 1350 500 50  0001 C CNN
+	1    6000 3000
+	0    1    1    0
+$EndComp
 $EndSCHEMATC
